File: PEP201-pojacavac klase A/PEP201-pojacavac klase A/PEP201-pojacavac klase A.kicad_pcb (KiCad board)
At the start: 2 copper layers, 45 x 45 mm, 28 parts, among them J1 Screw_Terminal_01x02, J3 Conn_01x02_Pin, Q1 MMBT2222A

Commit message: PEP201 prepared.
Parts:
- C1, C2, C3: footprint PEP_library:C_1206_3216Metric -> Capacitor_SMD:C_1206_3216Metric_Pad1.33x1.80mm_HandSolder
- R1, R2, R3, R4, R5: footprint PEP_library:R_smd_1206 -> Resistor_SMD:R_1206_3216Metric_Pad1.30x1.75mm_HandSolder
- moved REF** 20.0 mm to (113.5, 136.5)
- moved C3 7.34 mm to (129.0, 133.3)
- moved C2 3.18 mm to (131.8, 119.0), turned to 0 degrees
- moved J2 3.08 mm to (105.0, 118.0), turned to 180 degrees
- moved J4 2.98 mm to (140.0, 118.0), turned to 180 degrees
- moved R4 2.80 mm to (124.5, 130.3)
- moved C1 1.52 mm to (109.7, 119.0), turned to 0 degrees
- moved ? 1.10 mm to (131.6, 118.1)
- moved J1 0.80 mm to (122.2, 107.0)
- moved J5 0.44 mm to (140.0, 127.0)
- moved J3 0.28 mm to (105.0, 127.0)
- renumbered + to J2, + to J4, - to J5
Connections:
- C3 pad 1: 0 -> Net-(C3-Pad1)
- C3 pad 2: Net-(C3-Pad2) -> 0
- R5 pad 2: Net-(C3-Pad2) -> Net-(C3-Pad1)
Routing:
- net Net-(C3-Pad2): track 4.53 -> 0.00 mm
- net Tp1: track 13.9 -> 9.70 mm
- net 0: track 0.00 -> 3.89 mm, vias 0 -> 112
- net Net-(Q1-E): track 10.8 -> 13.4 mm
- net Net-(C3-Pad1): track 0.00 -> 2.45 mm
- net Net-(Q1-B): track 16.5 -> 14.8 mm
- net Net-(Q1-C): track 13.0 -> 12.1 mm
- net (no net): vias 109 -> 0
- added copper zone on B.Cu, net 0
- removed copper zone on F.Cu, net 0
Other:
- board text added: "+"
