File: PEP201-pojacavac klase A/PEP201-pojacavac klase A/PEP201-pojacavac klase A.kicad_sch (KiCad schematic)
At the start: 18 parts, among them J1 Screw_Terminal_01x02, J2 Conn_01x02_Pin, J3 Conn_01x02_Pin, J4 Conn_01x02_Pin, J5 Conn_01x02_Pin, Q1 MMBT2222A

Commit message: PEP201 prepared.
Parts:
- removed C1, C2, C3: 10u, PEP_library:C_1206_3216Metric, symbol GRT31CR61H106KE01L:GRT31CR61H106KE01L
- added C1, C2, C3: 10u, Capacitor_SMD:C_1206_3216Metric_Pad1.33x1.80mm_HandSolder, symbol Device:C
- R1, R2, R3, R4, R5: footprint PEP_library:R_smd_1206 -> Resistor_SMD:R_1206_3216Metric_Pad1.30x1.75mm_HandSolder
Connections:
- net 0: now also C3.2
- net Input signal: now also C1.1
- net Tp1: now also C2.2
- net at Q1.3 (C), R3.2: now also C2.1
- net at Q1.1 (B), R1.1, R2.1: now also C1.2
- net at R5.2: now also C3.1
Other:
- moved on the sheet: J2, J3, J4, J5
