File: PEP204-V1-differencijalni_par/PEP204-V1-differencijalni_par.kicad_pcb (KiCad board)
At the start: 2 copper layers, 45 x 45 mm, 25 parts, among them J1 Screw_Terminal_01x02, J2 Conn_01x02_Pin, J3 Conn_01x02_Pin, J4 Conn_01x02_Pin, J5 Conn_01x02_Pin, Q1 MMBT2222A, Q2 MMBT2222A, Q3 MMBT2222A, U1 CJ432

Commit message: PEP201 i PEP204 :)
Parts:
- removed the TP2 at (114.4, 118.2)
- removed the TP2 at (130.6, 118.2)
- added ?: , clipboard:5e84f11e-c99f-4f49-a7a0-7391ce06634b, F.Cu at (113.1, 133.2)
- added ?: , clipboard:997e7b5a-d5a8-41f9-879b-f51d86b09391, F.Cu at (130.1, 110.3)
- added ?: , clipboard:997e7b5a-d5a8-41f9-879b-f51d86b09391, F.Cu at (113.9, 110.3)
- added C1: 10u, PEP_library:C_1206_3216Metric, F.Cu at (122.5, 127.0)
- added J6: Conn_01x02_Pin, PEP_library:PinHeader_1x02_P2.54mm_Vertical, F.Cu at (104.8, 121.2)
- added J7: Conn_01x02_Pin, PEP_library:PinHeader_1x02_P2.54mm_Vertical, F.Cu at (140.3, 121.2)
- moved Q1 7.43 mm to (111.0, 121.5)
- moved Q3 7.42 mm to (134.0, 121.5)
- moved J2 7.14 mm to (104.7, 130.1)
- moved J3 7.06 mm to (140.3, 130.1)
- moved J4 7.06 mm to (140.3, 114.9)
- moved J5 7.01 mm to (104.7, 114.9)
- moved Q2 4.68 mm to (126.0, 126.9)
- moved U1 4.39 mm to (119.0, 126.9)
- moved ? 4.24 mm to (117.2, 135.2), turned to 90 degrees
- moved R1 3.97 mm to (114.8, 117.2), turned to 180 degrees
- moved R2 3.93 mm to (130.2, 117.2), turned to 0 degrees
- moved ? 3.62 mm to (106.7, 120.4)
- moved R4 3.18 mm to (115.5, 126.3)
- moved R3 3.18 mm to (129.4, 126.3), turned to 90 degrees
- moved TP2 1.75 mm to (122.5, 119.8)
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- renumbered R2 to R1, R5 to R2
Connections:
- net Net-(Q1-E) renamed Ve
- net Net-(Q2-B) renamed Vb
- J1 pad 1: GND -> 0
- J2 pad 2: GND -> Net-(J2-Pin_1)
- J3 pad 2: GND -> Net-(J3-Pin_1)
- J4 pad 2: GND -> Net-(J4-Pin_1)
- J5 pad 2: GND -> Net-(J5-Pin_1)
Routing:
- net Ve: track 13.6 -> 60.4 mm
- net Vcc: track 58.8 -> 30.1 mm
- net Net-(J3-Pin_1): track 7.77 -> 15.8 mm
- net Net-(J2-Pin_1): track 6.89 -> 14.3 mm
- net Vb: track 12.4 -> 5.88 mm
- net Net-(Q2-E): track 6.55 -> 2.62 mm
- net Net-(J4-Pin_1): track 18.9 -> 17.2 mm
- net Net-(U1-K): track 11.9 -> 13.2 mm
Other:
- board text added: "C1"
- board text added: "J1"
- board text added: "J2"
- board text added: "J3"
- board text added: "J4"
- board text added: "J5"
- board text added: "J6"
- board text added: "J7"
- board text added: "PEP204"
- board text added: "Q1"
- board text added: "Q2"
- board text added: "Q3"
- board text added: "R1"
- board text added: "R2"
- board text added: "R3"
- board text added: "R4"
- board text added: "RV1"
- board text added: "TP Ve"
- board text added: "TP Vout1"
- board text added: "TP Vout2"
- board text added: "U1"
- board text added: "Vin1"
- board text added: "Vin2"
- board text added: "Vout1"
- board text added: "Vout2"
- board text removed: "TP"
- board text removed: "Vi1"
- board text removed: "Vi2"
- board text removed: "Vu1"
- board text removed: "Vu2"

Commit message: PEP204 prepared.
Parts:
- removed TP2: TP Ve, TestPoint:TestPoint_Pad_D2.5mm
- added C2: 10u, PEP_library:C_1206_3216Metric, F.Cu at (122.2, 114.0)
- RV1: value R_Potentiometer -> 10k
- moved C1 10.9 mm to (115.6, 135.4), turned to -90 degrees
- moved U1 10.5 mm to (112.4, 135.1), turned to -90 degrees
- moved R3 8.07 mm to (124.6, 132.8), turned to -90 degrees
- moved RV1 5.31 mm to (119.7, 138.0)
- moved R1 4.73 mm to (114.3, 112.5), turned to -90 degrees
- moved R2 4.72 mm to (130.6, 112.5), turned to -90 degrees
- moved Q1 4.33 mm to (114.3, 118.7)
- moved Q3 4.00 mm to (131.1, 118.8)
- moved J1 3.86 mm to (122.2, 107.0)
- moved Q2 3.76 mm to (122.3, 127.6)
- moved R4 3.05 mm to (115.6, 129.4)
- moved J7 0.35 mm to (140.0, 121.2)
- moved J3 0.30 mm to (140.0, 130.1)
- moved J4 0.30 mm to (140.0, 114.9)
- moved J2 0.30 mm to (105.0, 130.1)
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Connections:
- net Vb renamed /Vb
- net Ve renamed /Ve
- J1 pad 1: 0 -> Vcc
- J1 pad 2: Vcc -> 0
Routing:
- net Vcc: track 30.1 -> 73.2 mm
- net /Ve: track 60.4 -> 21.6 mm
- net Net-(J2-Pin_1): track 14.3 -> 19.4 mm
- net GND: track 0.00 -> 4.91 mm, vias 0 -> 4
- net Net-(J3-Pin_1): track 15.8 -> 20.4 mm
- net /Vb: track 5.88 -> 10.2 mm
- net Net-(J5-Pin_1): track 17.1 -> 18.6 mm
- net Net-(Q2-E): track 2.62 -> 3.14 mm
- added copper zone on B.Cu, net GND
- removed copper zone on F.Cu, net GND
Other:
- board text added: "V_{in+}"
- board text added: "V_{in-}"
- board text added: "V_{out+}"
- board text added: "V_{out-}"
- board text removed: "C1"
- board text removed: "J1"
- board text removed: "J2"
- board text removed: "J3"
- board text removed: "J4"
- board text removed: "J5"
- board text removed: "J6"
- board text removed: "J7"
- board text removed: "Q1"
- board text removed: "Q2"
- board text removed: "Q3"
- board text removed: "R1"
- board text removed: "R2"
- board text removed: "R3"
- board text removed: "R4"
- board text removed: "RV1"
- board text removed: "TP Ve"
- board text removed: "TP Vout1"
- board text removed: "TP Vout2"
- board text removed: "U1"
- board text removed: "Vin1"
- board text removed: "Vin2"
- board text removed: "Vout1"
- board text removed: "Vout2"
