File: 90x90_template/90x90_template.kicad_pcb (KiCad board)
At the start: 2 copper layers, 90 x 90 mm, 41 parts, among them J1 Screw_Terminal_01x02

Commit message: Edge vias 0.
Merge attempt.
Routing:
- net 0: vias 0 -> 236
- net (no net): vias 236 -> 0
