File: 45x45_template/45x45_template.kicad_pcb (KiCad board)
At the start: 2 copper layers, 45 x 45 mm, 9 parts, among them J1 Screw_Terminal_01x02

Commit message: improved_templates
Routing:
- added copper zone on F.Cu, net 0
