File: 45x45_template/45x45_template.kicad_sch (KiCad schematic)
At the start: 8 parts, among them J1 Screw_Terminal_01x02

Commit message: fork
Parts:
- removed R1: 1Meg, PEP_library:R_Axial_DIN0207_L6.3mm_D2.5mm_P15.24mm_Horizontal, symbol PEP_library:R_THT
- removed TP1, TP2: TestPoint, symbol Connector:TestPoint
- added C1: 100u, symbol Device:C
- added C2, C3: 10u, symbol Device:C
- added J2, J3, J4, J5: Conn_01x02_Pin, Connector_PinHeader_2.54mm:PinHeader_1x02_P2.54mm_Vertical, symbol Connector:Conn_01x02_Pin
- added Q1: NPN, symbol Simulation_SPICE:NPN
- added R1, R2: 10k, symbol Device:R
- added R3: 4k7, symbol Device:R
Connections:
- net 0: now also J3.1 (Pin_1), J3.2 (Pin_2), J5.1 (Pin_1), J5.2 (Pin_2)
- net Input voltage renamed Vcc
- net Vcc: now also C1.1, Q1.1 (C), R1.1
- new net: C3.2, Q1.2 (B), R1.2, R2.1
- new net: C2.1, Q1.3 (E), R3.1
- new net GND: C1.2, R2.2, R3.2
- new net Input signal: C3.1, J2.1 (Pin_1), J2.2 (Pin_2)
- new net Tp1: C2.2, J4.1 (Pin_1), J4.2 (Pin_2)
Other:
- note added: "Konektori za ulazni signal"
- note added: "Pojačavač"
- note added: "Test point za osc"
- note removed: "Testpoint za merenje sa multimetrom"
- title: MegaOtpornik u vazduhu -> Emitter follower
- moved on the sheet: J1
