File: 45x90_template/45x90_template.kicad_pcb (KiCad board)
At the start: 2 copper layers, 90 x 45 mm, 41 parts, among them J1 Screw_Terminal_01x02

Commit message: improved_templates
Routing:
- net 0: vias 170 -> 169
- added copper zone on F.Cu, net 0
