File: PEP201-pojacavac_klase_A/PEP201-pojacavac_klase_A.kicad_pcb (KiCad board)
At the start: 2 copper layers, 45 x 45 mm, 28 parts, among them J1 Screw_Terminal_01x02, J2 Conn_01x02_Pin, J3 Conn_01x02_Pin, J4 Conn_01x02_Pin, J5 Conn_01x02_Pin, Q1 MMBT2222A

Commit message: Nova estetika.
Parts:
- removed the ? at (131.6, 118.1)
- removed the ? at (116.9, 109.8)
- removed the ? at (116.9, 123.0)
- removed the ? at (114.0, 121.2)
- removed the ? at (123.5, 123.0)
- removed the ? at (130.0, 124.2)
- added REF**: R_silk_symbol, PEP_library:R_silk_symbol, F.Cu at (117.1, 112.5)
- added REF**: C_silk_symbol, PEP_library:C_silk_symbol, F.Cu at (130.0, 126.5)
- added REF**: C_silk_symbol, PEP_library:C_silk_symbol, F.Cu at (129.8, 116.7)
- added REF**: R_silk_symbol, PEP_library:R_silk_symbol, F.Cu at (123.5, 126.7)
- added REF**: C_silk_symbol, PEP_library:C_silk_symbol, F.Cu at (113.9, 121.2)
- added REF**: R_silk_symbol, PEP_library:R_silk_symbol, F.Cu at (117.1, 126.3)
- moved ? 1.40 mm to (123.5, 107.1)
