File: PEP204-differencijalni_par/PEP204-differencijalni_par.kicad_pcb (KiCad board)
At the start: 2 copper layers, 45 x 45 mm, 29 parts, among them J1 Screw_Terminal_01x02, J2 Conn_01x02_Pin, J3 Conn_01x02_Pin, J4 Conn_01x02_Pin, J5 Conn_01x02_Pin, J6 Conn_01x02_Pin, J7 Conn_01x02_Pin, Q1 MMBT2222A, Q2 MMBT2222A, Q3 MMBT2222A, U1 CJ432

Commit message: ESTETIKKAA.
Parts:
- moved ? 10.7 mm to (113.4, 128.7)
- moved ? 2.96 mm to (113.9, 136.0)
- moved ? 2.63 mm to (115.8, 108.5)
- moved ? 2.28 mm to (117.2, 132.9)
- moved ? 1.80 mm to (130.1, 108.5)
Other:
- board text added: "V_{cc}"
