File: PEP202-emitter_follower/PEP202-emitter_follower.kicad_pcb (KiCad board)
At the start: 2 copper layers, 45 x 45 mm, 9 parts, among them J1 Screw_Terminal_01x02

Commit message: fork
Parts:
- removed REF**: ele_petnica_logo, PEP_library:ele_petnica_logo
- removed TP2 (x2): TestPoint, TestPoint:TestPoint_Pad_D2.5mm
- added C2: 10u, PEP_library:C_1206_3216Metric, F.Cu at (133.5, 126.5)
- added C3: 10u, PEP_library:C_1206_3216Metric, F.Cu at (113.0, 124.0)
- added J2: Conn_01x02_Pin, Connector_PinHeader_2.54mm:PinHeader_1x02_P2.54mm_Vertical, F.Cu at (105.0, 118.0)
- added J3: Conn_01x02_Pin, Connector_PinHeader_2.54mm:PinHeader_1x02_P2.54mm_Vertical, F.Cu at (105.0, 127.0)
- added J4: Conn_01x02_Pin, Connector_PinHeader_2.54mm:PinHeader_1x02_P2.54mm_Vertical, F.Cu at (140.0, 118.0)
- added J5: Conn_01x02_Pin, Connector_PinHeader_2.54mm:PinHeader_1x02_P2.54mm_Vertical, F.Cu at (140.0, 127.0)
- added Q1: NPN, Package_TO_SOT_SMD:SOT-23, F.Cu at (128.0, 126.0)
- added R2: 10k, PEP_library:R_smd_1206, F.Cu at (120.0, 131.5)
- added R3: 4k7, PEP_library:R_smd_1206, F.Cu at (128.0, 131.5)
- R1: value 1Meg -> 10k; footprint PEP_library:R_Axial_DIN0207_L6.3mm_D2.5mm_P15.24mm_Horizontal -> PEP_library:R_smd_1206
- moved R1 5.80 mm to (120.0, 120.5), turned to -90 degrees
Connections:
- J1 pad 1: Input voltage -> Vcc
- R1 pad 1: Net-(R1-Pad1) -> Vcc
- R1 pad 2: Input voltage -> Net-(Q1-B)
Routing:
- net 0: track 36.9 -> 0.00 mm, vias 0 -> 109
- net Net-(Q1-B): track 0.00 -> 21.7 mm
- net Vcc: track 0.00 -> 21.1 mm
- net Net-(R1-Pad1): track 13.9 -> 0.00 mm
- net Input voltage: track 11.5 -> 0.00 mm
- net Output signal: track 0.00 -> 8.04 mm
- net GND: track 0.00 -> 8.00 mm
- net Input signal: track 0.00 -> 7.96 mm
- net Net-(Q1-E): track 0.00 -> 7.63 mm
- net (no net): vias 109 -> 0
- added copper zone on B.Cu, net 0
Other:
- board text added: "Emitter-follower"
- board text removed: "MegaOtpornik u vazduhu"
