File: PEP202-emitter_follower/PEP202-emitter_follower.kicad_sch (KiCad schematic)
At the start: 8 parts, among them J1 Screw_Terminal_01x02

Commit message: fork
Parts:
- removed R1: 1Meg, PEP_library:R_Axial_DIN0207_L6.3mm_D2.5mm_P15.24mm_Horizontal, symbol PEP_library:R_THT
- removed TP1, TP2: TestPoint, symbol Connector:TestPoint
- added C2, C3: 10u, PEP_library:C_1206_3216Metric, symbol Device:C
- added J2, J3, J4, J5: Conn_01x02_Pin, Connector_PinHeader_2.54mm:PinHeader_1x02_P2.54mm_Vertical, symbol Connector:Conn_01x02_Pin
- added Q1: NPN, Package_TO_SOT_SMD:SOT-23, symbol Simulation_SPICE:NPN
- added R1, R2: 10k, PEP_library:R_smd_1206, symbol Device:R
- added R3: 4k7, PEP_library:R_smd_1206, symbol Device:R
Connections:
- net 0: now also J3.1 (Pin_1), J3.2 (Pin_2), J5.1 (Pin_1), J5.2 (Pin_2)
- net Input voltage renamed Vcc
- net Vcc: now also Q1.1 (C), R1.1
- new net: C3.2, Q1.2 (B), R1.2, R2.1
- new net: C2.1, Q1.3 (E), R3.1
- new net GND: R2.2, R3.2
- new net Input signal: C3.1, J2.1 (Pin_1), J2.2 (Pin_2)
- new net Output signal: C2.2, J4.1 (Pin_1), J4.2 (Pin_2)
Other:
- note added: "Konektor za izlazni signal"
- note added: "Konektori za ulazni signal"
- note added: "Pojačavač"
- note removed: "Testpoint za merenje sa multimetrom"
- title: MegaOtpornik u vazduhu -> Emitter follower
- moved on the sheet: J1
