File: PEP003-V1-redna_i_paralelna_otpornost/PEP003-V1-redna_i_paralelna_otpornost.kicad_pcb (KiCad board)
At the start: 2 copper layers, 90 x 45 mm, 41 parts, among them J1 Screw_Terminal_01x02

Commit message: lll
Parts:
- moved REF** 0.75 mm to (176.2, 72.8)
- moved REF** 0.75 mm to (176.2, 80.5)
- moved REF** 0.75 mm to (176.2, 87.5)
- moved REF** 0.75 mm to (176.2, 95.0)
- moved REF** 0.54 mm to (139.5, 68.5)
- moved REF** 0.54 mm to (139.5, 78.1)
- moved REF** 0.50 mm to (139.5, 90.1)
- moved REF** 0.44 mm to (139.5, 99.6)
