File: PEP005-V1-dzulov_zakon/PEP005-V1-dzulov_zakon.kicad_pcb (KiCad board)
At the start: 2 copper layers, 45 x 45 mm, 14 parts, among them J1 Conn_01x01_Socket, J2 Screw_Terminal_01x02, J3 Conn_01x01_Socket

Commit message: lll
Parts:
- moved G*** 3.25 mm to (142.5, 78.2)
- moved R3 2.00 mm to (131.9, 88.5)
- moved R2 1.75 mm to (131.9, 81.8)
- moved R1 1.50 mm to (131.9, 75.0)
- moved R4 1.50 mm to (131.9, 94.5)
- moved REF** 1.39 mm to (126.9, 69.5)
- moved REF** 1.25 mm to (143.0, 88.2)
Other:
- board text added: "10k"
