File: PEP006-V1-strujni_sant/PEP006-V1-strujni_sant.kicad_pcb (KiCad board)
At the start: 2 copper layers, 45 x 45 mm, 23 parts, among them J1 Screw_Terminal_01x02

Commit message: lll
Parts:
- moved REF** 34.7 mm to (138.2, 131.0)
- moved REF** 4.74 mm to (133.0, 128.8)
- moved REF** 4.74 mm to (126.0, 128.8)
- moved REF** 4.74 mm to (119.0, 128.8)
