File: PEP008-V1-RC_vremenska_konstanta/PEP008-V1-RC_vremenska_konstanta.kicad_pcb (KiCad board)
At the start: 2 copper layers, 45 x 45 mm, 20 parts, among them J1 Conn_01x01_Pin, J2 Screw_Terminal_01x02, J3 Conn_01x01_Pin, J4 Conn_01x01_Pin, J5 Conn_01x01_Pin, J6 Conn_01x03_Pin, J7 Conn_01x03_Pin, SW1 SW_SPDT, SW2 SW_SPDT

Commit message: lll
Parts:
- moved J6 1.00 mm to (140.0, 78.0)
Routing:
- net 0: track 40.3 -> 42.0 mm
- net Net-(J6-Pin_1): track 3.45 -> 4.46 mm
- net Net-(J6-Pin_3): track 3.48 -> 4.49 mm
- net Net-(J5-Pin_1): track 23.7 -> 22.7 mm
