File: PEP009-V1-LC_rezonantno_kolo/PEP009-V1-LC_rezonantno_kolo.kicad_pcb (KiCad board)
At the start: 2 copper layers, 45 x 45 mm, 22 parts, among them J1 Screw_Terminal_01x02, J2 Conn_01x01_Pin, J3 Conn_01x01_Pin, J4 Conn_01x01_Pin

Commit message: lll
Parts:
- moved REF** 1.34 mm to (147.1, 84.7)
- moved G*** 1.29 mm to (138.6, 84.2)
- moved REF** 0.90 mm to (147.0, 91.7)
- moved REF** 0.34 mm to (147.0, 98.7)
