File: PEP010-V1-Diode/PEP010-V1-Diode.kicad_pcb (KiCad board)
At the start: 2 copper layers, 45 x 45 mm, 32 parts, among them J1 Screw_Terminal_01x02, J2 Conn_01x01_Pin, J4 Conn_01x01_Pin, J5 Conn_01x01_Pin, J6 Conn_01x01_Pin, J7 Conn_01x01_Pin

Commit message: lll
Parts:
- removed D4: BZT52C5V1, PCM_JLCPCB:D_SOD-123
- added D5: D_Zener, Diode_THT:D_A-405_P7.62mm_Horizontal, F.Cu at (141.5, 70.6)
- moved G*** 34.1 mm to (123.8, 100.2)
- moved J4 1.75 mm to (120.5, 81.8)
- moved J5 1.75 mm to (126.8, 81.8)
- moved J6 1.75 mm to (133.5, 81.8)
- moved J7 1.75 mm to (141.5, 81.8)
- moved JP1 0.75 mm to (120.5, 94.0)
- moved JP2 0.75 mm to (126.8, 94.0)
- moved JP3 0.75 mm to (133.5, 94.0)
- moved JP4 0.75 mm to (141.5, 94.0)
- moved R1 0.75 mm to (120.5, 86.2)
- moved R2 0.75 mm to (126.8, 86.3)
- moved R3 0.75 mm to (133.5, 86.3)
- moved R4 0.75 mm to (141.5, 86.3)
Routing:
- net Net-(D5-A): track 9.51 -> 6.64 mm
- net Net-(D3-K): track 8.89 -> 9.64 mm
- net Net-(D2-K): track 9.56 -> 10.3 mm
- net Net-(D1-K): track 8.79 -> 9.54 mm
